File: hardware/gol.sch (EAGLE design)
At the start: 70 parts, among them J1 TC2050-IDC, J2 2057-MCR-B-S-RA-TSMT-NP-CS4-T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, U1 STM32F072CBT, U2 AP2111H-3.3TRG1SOT-223_DIO-M

Commit message: more routing
Connections:
- net EAST: now also U1A.PB10, U1A.PB11; no longer U1A.PA0, U1A.PA1
- net WEST: now also U1A.PA0, U1A.PA1; no longer U1A.PB10, U1A.PB11
Changed lines of the file:
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@@
 </segment>
 <segment>
-<pinref part="U1" gate="A" pin="PA1"/>
-<wire x1="45.72" y1="99.06" x2="43.18" y2="99.06" width="0.1524" layer="91"/>
-<wire x1="43.18" y1="99.06" x2="43.18" y2="101.6" width="0.1524" layer="91"/>
-<pinref part="U1" gate="A" pin="PA0"/>
-<wire x1="43.18" y1="101.6" x2="45.72" y2="101.6" width="0.1524" layer="91"/>
-<wire x1="43.18" y1="101.6" x2="40.64" y2="101.6" width="0.1524" layer="91"/>
-<junction x="43.18" y="101.6"/>
-<label x="40.64" y="101.6" size="1.27" layer="95" rot="R180" xref="yes"/>
+<label x="40.64" y="33.02" size="1.27" layer="95" rot="R180" xref="yes"/>
+<pinref part="U1" gate="A" pin="PB10"/>
+<wire x1="40.64" y1="33.02" x2="43.18" y2="33.02" width="0.1524" layer="91"/>
+<pinref part="U1" gate="A" pin="PB11"/>
+<wire x1="43.18" y1="33.02" x2="45.72" y2="33.02" width="0.1524" layer="91"/>
+<wire x1="45.72" y1="30.48" x2="43.18" y2="30.48" width="0.1524" layer="91"/>
+<wire x1="43.18" y1="30.48" x2="43.18" y2="33.02" width="0.1524" layer="91"/>
+<junction x="43.18" y="33.02"/>
 </segment>
 <segment>
@@
 </segment>
 <segment>
-<pinref part="U1" gate="A" pin="PB11"/>
-<wire x1="45.72" y1="30.48" x2="43.18" y2="30.48" width="0.1524" layer="91"/>
-<wire x1="43.18" y1="30.48" x2="43.18" y2="33.02" width="0.1524" layer="91"/>
-<pinref part="U1" gate="A" pin="PB10"/>
-<wire x1="43.18" y1="33.02" x2="45.72" y2="33.02" width="0.1524" layer="91"/>
-<wire x1="43.18" y1="33.02" x2="40.64" y2="33.02" width="0.1524" layer="91"/>
-<junction x="43.18" y="33.02"/>
-<label x="40.64" y="33.02" size="1.27" layer="95" rot="R180" xref="yes"/>
+<label x="40.64" y="101.6" size="1.27" layer="95" rot="R180" xref="yes"/>
+<pinref part="U1" gate="A" pin="PA0"/>
+<wire x1="40.64" y1="101.6" x2="43.18" y2="101.6" width="0.1524" layer="91"/>
+<pinref part="U1" gate="A" pin="PA1"/>
+<wire x1="43.18" y1="101.6" x2="45.72" y2="101.6" width="0.1524" layer="91"/>
+<wire x1="45.72" y1="99.06" x2="43.18" y2="99.06" width="0.1524" layer="91"/>
+<wire x1="43.18" y1="99.06" x2="43.18" y2="101.6" width="0.1524" layer="91"/>
+<junction x="43.18" y="101.6"/>
 </segment>
 <segment>

Commit message: more routing work
Connections:
- net OUTB-L2: now also U1A.PB12; no longer U1A.PA8
- net OUTB-L3: now also U1A.PA8; no longer U1A.PB12
Changed lines of the file:
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@@
 <segment>
 <pinref part="R5" gate="G$1" pin="2"/>
-<wire x1="12.7" y1="81.28" x2="12.7" y2="134.62" width="0.1524" layer="91"/>
+<wire x1="12.7" y1="30.48" x2="12.7" y2="134.62" width="0.1524" layer="91"/>
 <wire x1="12.7" y1="134.62" x2="33.02" y2="134.62" width="0.1524" layer="91"/>
-<pinref part="U1" gate="A" pin="PA8"/>
-<wire x1="12.7" y1="81.28" x2="45.72" y2="81.28" width="0.1524" layer="91"/>
+<wire x1="12.7" y1="30.48" x2="38.1" y2="30.48" width="0.1524" layer="91"/>
+<pinref part="U1" gate="A" pin="PB12"/>
+<wire x1="38.1" y1="30.48" x2="38.1" y2="27.94" width="0.1524" layer="91"/>
+<wire x1="38.1" y1="27.94" x2="45.72" y2="27.94" width="0.1524" layer="91"/>
 </segment>
 </net>
@@
 <segment>
 <pinref part="R6" gate="G$1" pin="2"/>
-<wire x1="10.16" y1="30.48" x2="10.16" y2="139.7" width="0.1524" layer="91"/>
+<wire x1="10.16" y1="81.28" x2="10.16" y2="139.7" width="0.1524" layer="91"/>
 <wire x1="10.16" y1="139.7" x2="33.02" y2="139.7" width="0.1524" layer="91"/>
-<pinref part="U1" gate="A" pin="PB12"/>
-<wire x1="45.72" y1="27.94" x2="35.56" y2="27.94" width="0.1524" layer="91"/>
-<wire x1="35.56" y1="27.94" x2="35.56" y2="30.48" width="0.1524" layer="91"/>
-<wire x1="35.56" y1="30.48" x2="10.16" y2="30.48" width="0.1524" layer="91"/>
+<pinref part="U1" gate="A" pin="PA8"/>
+<wire x1="45.72" y1="81.28" x2="10.16" y2="81.28" width="0.1524" layer="91"/>
 </segment>
 </net>
