File: hardware/gol.sch (EAGLE design)
At the start: 70 parts, among them J1 TC2050-IDC, J2 2057-MCR-B-S-RA-TSMT-NP-CS4-T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, U1 STM32F072CBT, U2 AP2111H-3.3TRG1SOT-223_DIO-M

Commit message: adds right-angle female header. replaces north with this.
Parts:
- BTN17: value BOOT -> FLASH
- NORTH: device pinhead:PINHD-1X4/90 -> parts:PINHD-1X041X04-RA-FEM
Changed lines of the file:
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@@
 <part name="R10" library="parts" deviceset="R-EU-0207/8" device=""/>
 <part name="SOUTH" library="pinhead" library_urn="urn:adsk.eagle:library:325" deviceset="PINHD-1X4" device="/90" package3d_urn="urn:adsk.eagle:package:22404/2" value="SOUTH"/>
-<part name="NORTH" library="pinhead" library_urn="urn:adsk.eagle:library:325" deviceset="PINHD-1X4" device="/90" package3d_urn="urn:adsk.eagle:package:22404/2" value="NORTH"/>
+<part name="NORTH" library="parts" deviceset="PINHD-1X04" device="1X04-RA-FEM" value="NORTH"/>
 <part name="GND3" library="supply1" library_urn="urn:adsk.eagle:library:371" deviceset="GND" device=""/>
 <part name="EAST" library="parts" deviceset="PINHD-1X04" device="" value="EAST"/>
@@
 <part name="R12" library="rcl" library_urn="urn:adsk.eagle:library:334" deviceset="R-EU_" device="R0603" package3d_urn="urn:adsk.eagle:package:23555/3" value="470k"/>
 <part name="GND6" library="supply1" library_urn="urn:adsk.eagle:library:371" deviceset="GND" device=""/>
-<part name="BTN17" library="parts" deviceset="BUTTON-RES" device="" value="BOOT"/>
+<part name="BTN17" library="parts" deviceset="BUTTON-RES" device="" value="FLASH"/>
 <part name="SUPPLY5" library="supply2" library_urn="urn:adsk.eagle:library:372" deviceset="V+" device=""/>
 <part name="BTN1" library="parts" deviceset="BUTTON-CAP" device=""/>
@@
 <attribute name="NAME" x="41.91" y="149.225" size="1.778" layer="95" rot="MR180"/>
 </instance>
-<instance part="NORTH" gate="A" x="12.7" y="154.94" smashed="yes" rot="MR0">
+<instance part="NORTH" gate="G$1" x="12.7" y="154.94" smashed="yes" rot="MR0">
 <attribute name="NAME" x="11.43" y="149.225" size="1.778" layer="95" rot="MR180"/>
 </instance>
@@
 </segment>
 <segment>
-<pinref part="NORTH" gate="A" pin="4"/>
+<pinref part="NORTH" gate="G$1" pin="4"/>
 <pinref part="SOUTH" gate="A" pin="1"/>
 <wire x1="15.24" y1="152.4" x2="27.94" y2="152.4" width="0.1524" layer="91"/>
@@
 <net name="CAN_TR" class="0">
 <segment>
-<pinref part="NORTH" gate="A" pin="2"/>
+<pinref part="NORTH" gate="G$1" pin="2"/>
 <pinref part="SOUTH" gate="A" pin="3"/>
 <wire x1="15.24" y1="157.48" x2="30.48" y2="157.48" width="0.1524" layer="91"/>
@@
 <net name="NORTH" class="0">
 <segment>
-<pinref part="NORTH" gate="A" pin="3"/>
+<pinref part="NORTH" gate="G$1" pin="3"/>
 <wire x1="15.24" y1="154.94" x2="20.32" y2="154.94" width="0.1524" layer="91"/>
 <label x="20.32" y="154.94" size="1.27" layer="95" xref="yes"/>
@@
 </segment>
 <segment>
-<pinref part="NORTH" gate="A" pin="1"/>
+<pinref part="NORTH" gate="G$1" pin="1"/>
 <pinref part="SOUTH" gate="A" pin="4"/>
 <wire x1="15.24" y1="160.02" x2="27.94" y2="160.02" width="0.1524" layer="91"/>

Commit message: Updates the mounting hole to take less floorspace.
Adds four mounting holes to the device. Rearranges some wires and vias to make it work.
Parts:
- added H1, H2, H3, H4: MOUNT-HOLE, parts:MOUNT-HOLE
Changed lines of the file:
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@@
 <grid distance="0.1" unitdist="inch" unit="inch" style="lines" multiple="1" display="no" altdistance="0.01" altunitdist="inch" altunit="inch"/>
 <layers>
-<layer number="1" name="Top" color="4" fill="1" visible="no" active="no"/>
-<layer number="16" name="Bottom" color="1" fill="1" visible="no" active="no"/>
-<layer number="17" name="Pads" color="2" fill="1" visible="no" active="no"/>
-<layer number="18" name="Vias" color="2" fill="1" visible="no" active="no"/>
-<layer number="19" name="Unrouted" color="6" fill="1" visible="no" active="no"/>
-<layer number="20" name="Dimension" color="24" fill="1" visible="no" active="no"/>
-<layer number="21" name="tPlace" color="7" fill="1" visible="no" active="no"/>
-<layer number="22" name="bPlace" color="7" fill="1" visible="no" active="no"/>
-<layer number="23" name="tOrigins" color="15" fill="1" visible="no" active="no"/>
-<layer number="24" name="bOrigins" color="15" fill="1" visible="no" active="no"/>
-<layer number="25" name="tNames" color="7" fill="1" visible="no" active="no"/>
-<layer number="26" name="bNames" color="7" fill="1" visible="no" active="no"/>
-<layer number="27" name="tValues" color="7" fill="1" visible="no" active="no"/>
-<layer number="28" name="bValues" color="7" fill="1" visible="no" active="no"/>
+<layer number="1" name="Top" color="4" fill="1" visible="yes" active="no"/>
+<layer number="16" name="Bottom" color="1" fill="1" visible="yes" active="no"/>
+<layer number="17" name="Pads" color="2" fill="1" visible="yes" active="no"/>
+<layer number="18" name="Vias" color="2" fill="1" visible="yes" active="no"/>
+<layer number="19" name="Unrouted" color="6" fill="1" visible="yes" active="no"/>
+<layer number="20" name="Dimension" color="24" fill="1" visible="yes" active="no"/>
+<layer number="21" name="tPlace" color="7" fill="1" visible="yes" active="no"/>
+<layer number="22" name="bPlace" color="7" fill="1" visible="yes" active="no"/>
+<layer number="23" name="tOrigins" color="15" fill="1" visible="yes" active="no"/>
+<layer number="24" name="bOrigins" color="15" fill="1" visible="yes" active="no"/>
+<layer number="25" name="tNames" color="7" fill="1" visible="yes" active="no"/>
+<layer number="26" name="bNames" color="7" fill="1" visible="yes" active="no"/>
+<layer number="27" name="tValues" color="7" fill="1" visible="yes" active="no"/>
+<layer number="28" name="bValues" color="7" fill="1" visible="yes" active="no"/>
 <layer number="29" name="tStop" color="7" fill="3" visible="no" active="no"/>
 <layer number="30" name="bStop" color="7" fill="6" visible="no" active="no"/>
@@
 <layer number="35" name="tGlue" color="7" fill="4" visible="no" active="no"/>
 <layer number="36" name="bGlue" color="7" fill="5" visible="no" active="no"/>
-<layer number="37" name="tTest" color="7" fill="1" visible="no" active="no"/>
-<layer number="38" name="bTest" color="7" fill="1" visible="no" active="no"/>
+<layer number="37" name="tTest" color="7" fill="1" visible="yes" active="no"/>
+<layer number="38" name="bTest" color="7" fill="1" visible="yes" active="no"/>
 <layer number="39" name="tKeepout" color="4" fill="11" visible="no" active="no"/>
 <layer number="40" name="bKeepout" color="1" fill="11" visible="no" active="no"/>
@@
 <layer number="44" name="Drills" color="7" fill="1" visible="no" active="no"/>
 <layer number="45" name="Holes" color="7" fill="1" visible="no" active="no"/>
-<layer number="46" name="Milling" color="3" fill="1" visible="no" active="no"/>
-<layer number="47" name="Measures" color="7" fill="1" visible="no" active="no"/>
-<layer number="48" name="Document" color="7" fill="1" visible="no" active="no"/>
-<layer number="49" name="Reference" color="7" fill="1" visible="no" active="no"/>
-<layer number="50" name="dxf" color="7" fill="1" visible="no" active="no"/>
-<layer number="51" name="tDocu" color="7" fill="1" visible="no" active="no"/>
-<layer number="52" name="bDocu" color="7" fill="1" visible="no" active="no"/>
-<layer number="53" name="tGND_GNDA" color="7" fill="9" visible="no" active="no"/>
-<layer number="54" name="bGND_GNDA" color="1" fill="9" visible="no" active="no"/>
-<layer number="56" name="wert" color="7" fill="1" visible="no" active="no"/>
+<layer number="46" name="Milling" color="3" fill="1" visible="yes" active="no"/>
+<layer number="47" name="Measures" color="7" fill="1" visible="yes" active="no"/>
+<layer number="48" name="Document" color="7" fill="1" visible="yes" active="no"/>
+<layer number="49" name="Reference" color="7" fill="1" visible="yes" active="no"/>
+<layer number="50" name="dxf" color="7" fill="1" visible="yes" active="no"/>
+<layer number="51" name="tDocu" color="7" fill="1" visible="yes" active="no"/>
+<layer number="52" name="bDocu" color="7" fill="1" visible="yes" active="no"/>
+<layer number="53" name="tGND_GNDA" color="7" fill="9" visible="yes" active="no"/>
+<layer number="54" name="bGND_GNDA" color="1" fill="9" visible="yes" active="no"/>
+<layer number="56" name="wert" color="7" fill="1" visible="yes" active="no"/>
 <layer number="88" name="SimResults" color="9" fill="1" visible="yes" active="yes"/>
 <layer number="89" name="SimProbes" color="9" fill="1" visible="yes" active="yes"/>
@@
 <part name="SUPPLY10" library="supply2" library_urn="urn:adsk.eagle:library:372" deviceset="+5V" device=""/>
 <part name="GND12" library="supply1" library_urn="urn:adsk.eagle:library:371" deviceset="GND" device=""/>
+<part name="H1" library="parts" deviceset="MOUNT-HOLE" device="" value="MOUNT-HOLE"/>
+<part name="H2" library="parts" deviceset="MOUNT-HOLE" device=""/>
+<part name="H3" library="parts" deviceset="MOUNT-HOLE" device=""/>
+<part name="H4" library="parts" deviceset="MOUNT-HOLE" device=""/>
 </parts>
 <sheets>
@@
 <attribute name="VALUE" x="66.04" y="144.78" size="1.778" layer="96"/>
 </instance>
+<instance part="H1" gate="G$1" x="114.3" y="33.02" smashed="yes">
+<attribute name="NAME" x="116.332" y="33.6042" size="1.778" layer="95"/>
+<attribute name="VALUE" x="116.332" y="30.5562" size="1.778" layer="96"/>
+</instance>
+<instance part="H2" gate="G$1" x="114.3" y="25.4" smashed="yes">
+<attribute name="NAME" x="116.332" y="25.9842" size="1.778" layer="95"/>
+<attribute name="VALUE" x="116.332" y="22.9362" size="1.778" layer="96"/>
+</instance>
+<instance part="H3" gate="G$1" x="114.3" y="17.78" smashed="yes">
+<attribute name="NAME" x="116.332" y="18.3642" size="1.778" layer="95"/>
+<attribute name="VALUE" x="116.332" y="15.3162" size="1.778" layer="96"/>
+</instance>
+<instance part="H4" gate="G$1" x="114.3" y="10.16" smashed="yes">
+<attribute name="NAME" x="116.332" y="10.7442" size="1.778" layer="95"/>
+<attribute name="VALUE" x="116.332" y="7.6962" size="1.778" layer="96"/>
+</instance>
 </instances>
