File: hardware/gol.sch (EAGLE design)
At the start: 74 parts, among them J1 TC2050-IDC, J2 2057-MCR-B-S-RA-TSMT-NP-CS4-T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, U1 STM32F072CBT, U2 AP2111H-3.3TRG1SOT-223_DIO-M

Commit message: Adds gerber and assembly files for prototype run. Adds missing values for the pnp render. Adds a rendered pdf schematic.
Parts:
- C1, C2, C3, C7, C8: value (none) -> 1 uF
Changed lines of the file:
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@@
 <part name="GND1" library="supply1" library_urn="urn:adsk.eagle:library:371" deviceset="GND" device=""/>
 <part name="SUPPLY1" library="supply2" library_urn="urn:adsk.eagle:library:372" deviceset="V+" device=""/>
-<part name="C1" library="rcl" library_urn="urn:adsk.eagle:library:334" deviceset="C-EU" device="C0603" package3d_urn="urn:adsk.eagle:package:23616/2"/>
-<part name="C2" library="rcl" library_urn="urn:adsk.eagle:library:334" deviceset="C-EU" device="C0603" package3d_urn="urn:adsk.eagle:package:23616/2"/>
-<part name="C3" library="rcl" library_urn="urn:adsk.eagle:library:334" deviceset="C-EU" device="C0603" package3d_urn="urn:adsk.eagle:package:23616/2"/>
+<part name="C1" library="rcl" library_urn="urn:adsk.eagle:library:334" deviceset="C-EU" device="C0603" package3d_urn="urn:adsk.eagle:package:23616/2" value="1 uF"/>
+<part name="C2" library="rcl" library_urn="urn:adsk.eagle:library:334" deviceset="C-EU" device="C0603" package3d_urn="urn:adsk.eagle:package:23616/2" value="1 uF"/>
+<part name="C3" library="rcl" library_urn="urn:adsk.eagle:library:334" deviceset="C-EU" device="C0603" package3d_urn="urn:adsk.eagle:package:23616/2" value="1 uF"/>
 <part name="SUPPLY2" library="supply2" library_urn="urn:adsk.eagle:library:372" deviceset="V+" device=""/>
 <part name="GND2" library="supply1" library_urn="urn:adsk.eagle:library:371" deviceset="GND" device=""/>
@@
 <part name="SUPPLY7" library="supply2" library_urn="urn:adsk.eagle:library:372" deviceset="+5V" device=""/>
 <part name="SUPPLY8" library="supply2" library_urn="urn:adsk.eagle:library:372" deviceset="+5V" device=""/>
-<part name="C7" library="rcl" library_urn="urn:adsk.eagle:library:334" deviceset="C-EU" device="C0603" package3d_urn="urn:adsk.eagle:package:23616/2"/>
+<part name="C7" library="rcl" library_urn="urn:adsk.eagle:library:334" deviceset="C-EU" device="C0603" package3d_urn="urn:adsk.eagle:package:23616/2" value="1 uF"/>
 <part name="GND10" library="supply1" library_urn="urn:adsk.eagle:library:371" deviceset="GND" device=""/>
 <part name="SUPPLY9" library="supply2" library_urn="urn:adsk.eagle:library:372" deviceset="V+" device=""/>
-<part name="C8" library="rcl" library_urn="urn:adsk.eagle:library:334" deviceset="C-EU" device="C0603" package3d_urn="urn:adsk.eagle:package:23616/2"/>
+<part name="C8" library="rcl" library_urn="urn:adsk.eagle:library:334" deviceset="C-EU" device="C0603" package3d_urn="urn:adsk.eagle:package:23616/2" value="1 uF"/>
 <part name="BTN19" library="parts" deviceset="BUTTON-RES" device="" value="RESET"/>
 <part name="GND11" library="supply1" library_urn="urn:adsk.eagle:library:371" deviceset="GND" device=""/>

Commit message: Moves the capacitive sensors from PB5-6 to PB6-7. Switches the debug output from PB7 to PB5.
Connections:
- removed net PB7: J1.7, U1A.PB7
- new net DBG1: J1.7, U1A.PB5
- net COL3: now also U1A.PB6; no longer U1A.PB5
- net ROW3: now also U1A.PB7; no longer U1A.PB6
Changed lines of the file:
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@@
 <grid distance="0.1" unitdist="inch" unit="inch" style="lines" multiple="1" display="no" altdistance="0.01" altunitdist="inch" altunit="inch"/>
 <layers>
-<layer number="1" name="Top" color="4" fill="1" visible="yes" active="no"/>
-<layer number="16" name="Bottom" color="1" fill="1" visible="yes" active="no"/>
-<layer number="17" name="Pads" color="2" fill="1" visible="yes" active="no"/>
-<layer number="18" name="Vias" color="2" fill="1" visible="yes" active="no"/>
-<layer number="19" name="Unrouted" color="6" fill="1" visible="yes" active="no"/>
-<layer number="20" name="Dimension" color="24" fill="1" visible="yes" active="no"/>
-<layer number="21" name="tPlace" color="7" fill="1" visible="yes" active="no"/>
-<layer number="22" name="bPlace" color="7" fill="1" visible="yes" active="no"/>
-<layer number="23" name="tOrigins" color="15" fill="1" visible="yes" active="no"/>
-<layer number="24" name="bOrigins" color="15" fill="1" visible="yes" active="no"/>
-<layer number="25" name="tNames" color="7" fill="1" visible="yes" active="no"/>
-<layer number="26" name="bNames" color="7" fill="1" visible="yes" active="no"/>
-<layer number="27" name="tValues" color="7" fill="1" visible="yes" active="no"/>
-<layer number="28" name="bValues" color="7" fill="1" visible="yes" active="no"/>
+<layer number="1" name="Top" color="4" fill="1" visible="no" active="no"/>
+<layer number="16" name="Bottom" color="1" fill="1" visible="no" active="no"/>
+<layer number="17" name="Pads" color="2" fill="1" visible="no" active="no"/>
+<layer number="18" name="Vias" color="2" fill="1" visible="no" active="no"/>
+<layer number="19" name="Unrouted" color="6" fill="1" visible="no" active="no"/>
+<layer number="20" name="Dimension" color="24" fill="1" visible="no" active="no"/>
+<layer number="21" name="tPlace" color="7" fill="1" visible="no" active="no"/>
+<layer number="22" name="bPlace" color="7" fill="1" visible="no" active="no"/>
+<layer number="23" name="tOrigins" color="15" fill="1" visible="no" active="no"/>
+<layer number="24" name="bOrigins" color="15" fill="1" visible="no" active="no"/>
+<layer number="25" name="tNames" color="7" fill="1" visible="no" active="no"/>
+<layer number="26" name="bNames" color="7" fill="1" visible="no" active="no"/>
+<layer number="27" name="tValues" color="7" fill="1" visible="no" active="no"/>
+<layer number="28" name="bValues" color="7" fill="1" visible="no" active="no"/>
 <layer number="29" name="tStop" color="7" fill="3" visible="no" active="no"/>
 <layer number="30" name="bStop" color="7" fill="6" visible="no" active="no"/>
@@
 <layer number="35" name="tGlue" color="7" fill="4" visible="no" active="no"/>
 <layer number="36" name="bGlue" color="7" fill="5" visible="no" active="no"/>
-<layer number="37" name="tTest" color="7" fill="1" visible="yes" active="no"/>
-<layer number="38" name="bTest" color="7" fill="1" visible="yes" active="no"/>
+<layer number="37" name="tTest" color="7" fill="1" visible="no" active="no"/>
+<layer number="38" name="bTest" color="7" fill="1" visible="no" active="no"/>
 <layer number="39" name="tKeepout" color="4" fill="11" visible="no" active="no"/>
 <layer number="40" name="bKeepout" color="1" fill="11" visible="no" active="no"/>
@@
 <layer number="44" name="Drills" color="7" fill="1" visible="no" active="no"/>
 <layer number="45" name="Holes" color="7" fill="1" visible="no" active="no"/>
-<layer number="46" name="Milling" color="3" fill="1" visible="yes" active="no"/>
-<layer number="47" name="Measures" color="7" fill="1" visible="yes" active="no"/>
-<layer number="48" name="Document" color="7" fill="1" visible="yes" active="no"/>
-<layer number="49" name="Reference" color="7" fill="1" visible="yes" active="no"/>
-<layer number="50" name="dxf" color="7" fill="1" visible="yes" active="no"/>
-<layer number="51" name="tDocu" color="7" fill="1" visible="yes" active="no"/>
-<layer number="52" name="bDocu" color="7" fill="1" visible="yes" active="no"/>
-<layer number="53" name="tGND_GNDA" color="7" fill="9" visible="yes" active="no"/>
-<layer number="54" name="bGND_GNDA" color="1" fill="9" visible="yes" active="no"/>
-<layer number="56" name="wert" color="7" fill="1" visible="yes" active="no"/>
+<layer number="46" name="Milling" color="3" fill="1" visible="no" active="no"/>
+<layer number="47" name="Measures" color="7" fill="1" visible="no" active="no"/>
+<layer number="48" name="Document" color="7" fill="1" visible="no" active="no"/>
+<layer number="49" name="Reference" color="7" fill="1" visible="no" active="no"/>
+<layer number="50" name="dxf" color="7" fill="1" visible="no" active="no"/>
+<layer number="51" name="tDocu" color="7" fill="1" visible="no" active="no"/>
+<layer number="52" name="bDocu" color="7" fill="1" visible="no" active="no"/>
+<layer number="53" name="tGND_GNDA" color="7" fill="9" visible="no" active="no"/>
+<layer number="54" name="bGND_GNDA" color="1" fill="9" visible="no" active="no"/>
+<layer number="56" name="wert" color="7" fill="1" visible="no" active="no"/>
 <layer number="88" name="SimResults" color="9" fill="1" visible="yes" active="yes"/>
 <layer number="89" name="SimProbes" color="9" fill="1" visible="yes" active="yes"/>
@@
 </segment>
 <segment>
-<pinref part="U1" gate="A" pin="PB5"/>
-<wire x1="45.72" y1="45.72" x2="40.64" y2="45.72" width="0.1524" layer="91"/>
-<label x="40.64" y="45.72" size="1.27" layer="95" rot="R180" xref="yes"/>
+<label x="40.64" y="43.18" size="1.27" layer="95" rot="R180" xref="yes"/>
+<pinref part="U1" gate="A" pin="PB6"/>
+<wire x1="40.64" y1="43.18" x2="45.72" y2="43.18" width="0.1524" layer="91"/>
 </segment>
 </net>
@@
 </segment>
 <segment>
-<pinref part="U1" gate="A" pin="PB6"/>
-<wire x1="45.72" y1="43.18" x2="40.64" y2="43.18" width="0.1524" layer="91"/>
-<label x="40.64" y="43.18" size="1.27" layer="95" rot="R180" xref="yes"/>
+<label x="40.64" y="40.64" size="1.27" layer="95" rot="R180" xref="yes"/>
+<pinref part="U1" gate="A" pin="PB7"/>
+<wire x1="40.64" y1="40.64" x2="45.72" y2="40.64" width="0.1524" layer="91"/>
 </segment>
 </net>
@@
 </segment>
 </net>
-<net name="PB7" class="0">
+<net name="DBG1" class="0">
 <segment>
 <wire x1="139.7" y1="147.32" x2="160.02" y2="147.32" width="0.1524" layer="91"/>
@@
 </segment>
 <segment>
-<pinref part="U1" gate="A" pin="PB7"/>
-<wire x1="45.72" y1="40.64" x2="40.64" y2="40.64" width="0.1524" layer="91"/>
-<label x="40.64" y="40.64" size="1.27" layer="95" rot="R180" xref="yes"/>
-</segment>
-</net>
+<wire x1="40.64" y1="45.72" x2="45.72" y2="45.72" width="0.1524" layer="91"/>
+<pinref part="U1" gate="A" pin="PB5"/>
+<label x="40.64" y="45.72" size="1.27" layer="95" rot="R180" xref="yes"/>
+</segment>
+</net>

Commit message: Replaces the menu button with capacitive option. Adds cirles and numbers to the capacitive buttons.
Parts:
- BTN1: value BUTTON-CAP -> 1
- BTN10: value BUTTON-CAP -> 10
- BTN11: value BUTTON-CAP -> 11
- BTN12: value BUTTON-CAP -> 12
- BTN13: value BUTTON-CAP -> 13
- BTN14: value BUTTON-CAP -> 14
- BTN15: value BUTTON-CAP -> 15
- BTN16: value BUTTON-CAP -> 16
- BTN18: device parts:BUTTON-RES -> parts:BUTTON-CAPNARROW
- BTN2: value BUTTON-CAP -> 2
- BTN3: value BUTTON-CAP -> 3
- BTN4: value BUTTON-CAP -> 4
- BTN5: value BUTTON-CAP -> 5
- BTN6: value BUTTON-CAP -> 6
- BTN7: value BUTTON-CAP -> 7
- BTN8: value BUTTON-CAP -> 8
- BTN9: value BUTTON-CAP -> 9
Connections:
- removed net PB15: BTN18.2, J1.5, U1A.PB15
- new net DBG2: J1.5, U1A.PB15
- net GND: no longer BTN18.1
- net IN_ROW0: now also BTN18.1
- net IN_ROW2: now also BTN18.2
Changed lines of the file:
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@@
 <part name="BTN17" library="parts" deviceset="BUTTON-RES" device="" value="FLASH"/>
 <part name="SUPPLY5" library="supply2" library_urn="urn:adsk.eagle:library:372" deviceset="V+" device=""/>
-<part name="BTN1" library="parts" deviceset="BUTTON-CAP" device=""/>
-<part name="BTN2" library="parts" deviceset="BUTTON-CAP" device=""/>
-<part name="BTN3" library="parts" deviceset="BUTTON-CAP" device=""/>
-<part name="BTN4" library="parts" deviceset="BUTTON-CAP" device=""/>
-<part name="BTN5" library="parts" deviceset="BUTTON-CAP" device=""/>
-<part name="BTN6" library="parts" deviceset="BUTTON-CAP" device=""/>
-<part name="BTN7" library="parts" deviceset="BUTTON-CAP" device=""/>
-<part name="BTN8" library="parts" deviceset="BUTTON-CAP" device=""/>
-<part name="BTN9" library="parts" deviceset="BUTTON-CAP" device=""/>
-<part name="BTN10" library="parts" deviceset="BUTTON-CAP" device=""/>
-<part name="BTN11" library="parts" deviceset="BUTTON-CAP" device=""/>
-<part name="BTN12" library="parts" deviceset="BUTTON-CAP" device=""/>
-<part name="BTN13" library="parts" deviceset="BUTTON-CAP" device=""/>
-<part name="BTN14" library="parts" deviceset="BUTTON-CAP" device=""/>
-<part name="BTN15" library="parts" deviceset="BUTTON-CAP" device=""/>
-<part name="BTN16" library="parts" deviceset="BUTTON-CAP" device=""/>
-<part name="BTN18" library="parts" deviceset="BUTTON-RES" device="" value="MENU"/>
-<part name="GND7" library="supply1" library_urn="urn:adsk.eagle:library:371" deviceset="GND" device=""/>
+<part name="BTN1" library="parts" deviceset="BUTTON-CAP" device="" value="1"/>
+<part name="BTN2" library="parts" deviceset="BUTTON-CAP" device="" value="2"/>
+<part name="BTN3" library="parts" deviceset="BUTTON-CAP" device="" value="3"/>
+<part name="BTN4" library="parts" deviceset="BUTTON-CAP" device="" value="4"/>
+<part name="BTN5" library="parts" deviceset="BUTTON-CAP" device="" value="5"/>
+<part name="BTN6" library="parts" deviceset="BUTTON-CAP" device="" value="6"/>
+<part name="BTN7" library="parts" deviceset="BUTTON-CAP" device="" value="7"/>
+<part name="BTN8" library="parts" deviceset="BUTTON-CAP" device="" value="8"/>
+<part name="BTN9" library="parts" deviceset="BUTTON-CAP" device="" value="9"/>
+<part name="BTN10" library="parts" deviceset="BUTTON-CAP" device="" value="10"/>
+<part name="BTN11" library="parts" deviceset="BUTTON-CAP" device="" value="11"/>
+<part name="BTN12" library="parts" deviceset="BUTTON-CAP" device="" value="12"/>
+<part name="BTN13" library="parts" deviceset="BUTTON-CAP" device="" value="13"/>
+<part name="BTN14" library="parts" deviceset="BUTTON-CAP" device="" value="14"/>
+<part name="BTN15" library="parts" deviceset="BUTTON-CAP" device="" value="15"/>
+<part name="BTN16" library="parts" deviceset="BUTTON-CAP" device="" value="16"/>
+<part name="BTN18" library="parts" deviceset="BUTTON-CAP" device="NARROW" value="MENU"/>
 <part name="R11" library="rcl" library_urn="urn:adsk.eagle:library:334" deviceset="R-EU_" device="R0603" package3d_urn="urn:adsk.eagle:package:23555/3" value="10k"/>
 <part name="R13" library="rcl" library_urn="urn:adsk.eagle:library:334" deviceset="R-EU_" device="R0603" package3d_urn="urn:adsk.eagle:package:23555/3" value="10k"/>
@@
 <attribute name="NAME" x="236.22" y="40.64" size="1.778" layer="95"/>
 </instance>
-<instance part="BTN18" gate="G$1" x="30.48" y="10.16" smashed="yes">
-<attribute name="NAME" x="27.94" y="12.7" size="1.778" layer="95"/>
-</instance>
-<instance part="GND7" gate="1" x="7.62" y="7.62" smashed="yes">
-<attribute name="VALUE" x="5.08" y="5.08" size="1.778" layer="96"/>
+<instance part="BTN18" gate="G$1" x="251.46" y="53.34" smashed="yes" rot="R270">
+<attribute name="NAME" x="254" y="55.88" size="1.778" layer="95" rot="R270"/>
 </instance>
 <instance part="R11" gate="G$1" x="172.72" y="81.28" smashed="yes" rot="R270">
@@
 </segment>
 <segment>
-<pinref part="GND7" gate="1" pin="GND"/>
-<pinref part="BTN18" gate="G$1" pin="1"/>
-<wire x1="7.62" y1="10.16" x2="25.4" y2="10.16" width="0.1524" layer="91"/>
-</segment>
-<segment>
 <wire x1="139.7" y1="157.48" x2="162.56" y2="157.48" width="0.1524" layer="91"/>
 <wire x1="162.56" y1="157.48" x2="162.56" y2="137.16" width="0.1524" layer="91"/>
@@
 <wire x1="205.74" y1="63.5" x2="223.52" y2="63.5" width="0.1524" layer="91"/>
 <wire x1="223.52" y1="63.5" x2="241.3" y2="63.5" width="0.1524" layer="91"/>
-<wire x1="241.3" y1="63.5" x2="246.38" y2="63.5" width="0.1524" layer="91"/>
 <wire x1="185.42" y1="68.58" x2="187.96" y2="68.58" width="0.1524" layer="91"/>
 <wire x1="187.96" y1="68.58" x2="187.96" y2="63.5" width="0.1524" layer="91"/>
@@
 <wire x1="187.96" y1="63.5" x2="170.18" y2="63.5" width="0.1524" layer="91"/>
 <junction x="187.96" y="63.5"/>
+<wire x1="241.3" y1="63.5" x2="251.46" y2="63.5" width="0.1524" layer="91"/>
+<pinref part="BTN18" gate="G$1" pin="1"/>
+<wire x1="251.46" y1="63.5" x2="251.46" y2="58.42" width="0.1524" layer="91"/>
 </segment>
 </net>
@@
 <wire x1="205.74" y1="43.18" x2="223.52" y2="43.18" width="0.1524" layer="91"/>
 <wire x1="223.52" y1="43.18" x2="241.3" y2="43.18" width="0.1524" layer="91"/>
-<wire x1="241.3" y1="43.18" x2="246.38" y2="43.18" width="0.1524" layer="91"/>
 <wire x1="185.42" y1="48.26" x2="187.96" y2="48.26" width="0.1524" layer="91"/>
 <wire x1="187.96" y1="48.26" x2="187.96" y2="43.18" width="0.1524" layer="91"/>
@@
 <wire x1="187.96" y1="43.18" x2="170.18" y2="43.18" width="0.1524" layer="91"/>
 <junction x="187.96" y="43.18"/>
+<wire x1="241.3" y1="43.18" x2="251.46" y2="43.18" width="0.1524" layer="91"/>
+<pinref part="BTN18" gate="G$1" pin="2"/>
+<wire x1="251.46" y1="43.18" x2="251.46" y2="48.26" width="0.1524" layer="91"/>
 </segment>
 </net>
@@
 </segment>
 </net>
-<net name="PB15" class="0">
+<net name="DBG2" class="0">
 <segment>
 <wire x1="139.7" y1="152.4" x2="160.02" y2="152.4" width="0.1524" layer="91"/>
@@
 </segment>
 <segment>
-<pinref part="BTN18" gate="G$1" pin="2"/>
-<wire x1="35.56" y1="10.16" x2="38.1" y2="10.16" width="0.1524" layer="91"/>
-<wire x1="38.1" y1="10.16" x2="38.1" y2="20.32" width="0.1524" layer="91"/>
 <pinref part="U1" gate="A" pin="PB15"/>
-<wire x1="38.1" y1="20.32" x2="45.72" y2="20.32" width="0.1524" layer="91"/>
-<label x="38.1" y="17.78" size="1.27" layer="95" xref="yes"/>
-</segment>
-</net>
+<wire x1="43.18" y1="20.32" x2="45.72" y2="20.32" width="0.1524" layer="91"/>
+<label x="43.18" y="20.32" size="1.27" layer="95" rot="R180" xref="yes"/>
+</segment>
+</net>
